File: Design Files/Kicad Files/Matrix Game.sch (KiCad schematic (older format))
At the start: 20 parts

Commit message: Reset switch added
Parts:
- added SW?: SW_PUSH, symbol SW_PUSH
- R?: value 100K -> 10k
Connections:
- net GND: now also SW?.2
- net at C?.2, IC?.1 ((PCINT14/~RESET~)PC6), R?.2: now also SW?.1
